Commit message: revised

File: urdf/KDARPA.urdf (robot description, URDF)
Before this commit: robot KDARPA, 33 links, 32 joints
Links:
- link base_Link: geometry collision mesh filename=package://kdarpa_world/meshes/base_Link.STL; visual mesh filename=package://kdarpa_world/meshes/base_Link.STL
- link front_door_link: geometry collision mesh filename=package://kdarpa_world/meshes/front_door_link.STL; visual mesh filename=package://kdarpa_world/meshes/front_door_link.STL
- link ground_in_Link: geometry collision mesh filename=package://kdarpa_world/meshes/ground_in_Link.STL; visual mesh filename=package://kdarpa_world/meshes/ground_in_Link.STL
- link ground_link: geometry collision mesh filename=package://kdarpa_world/meshes/ground_link.STL; visual mesh filename=package://kdarpa_world/meshes/ground_link.STL
- link handle_1_Link: geometry collision mesh filename=package://kdarpa_world/meshes/handle_1_Link.STL; visual mesh filename=package://kdarpa_world/meshes/handle_1_Link.STL
- link handle_2_Link: geometry collision mesh filename=package://kdarpa_world/meshes/handle_2_Link.STL; visual mesh filename=package://kdarpa_world/meshes/handle_2_Link.STL
- link handle_3_Link: geometry collision mesh filename=package://kdarpa_world/meshes/handle_3_Link.STL; visual mesh filename=package://kdarpa_world/meshes/handle_3_Link.STL
- link indoor_fence_Link: geometry collision mesh filename=package://kdarpa_world/meshes/indoor_fence_Link.STL; visual mesh filename=package://kdarpa_world/meshes/indoor_fence_Link.STL
- link open_window_Link: geometry collision mesh filename=package://kdarpa_world/meshes/open_window_Link.STL; visual mesh filename=package://kdarpa_world/meshes/open_window_Link.STL
- link outdoor_left_wall: geometry collision mesh filename=package://kdarpa_world/meshes/outdoor_left_wall.STL; visual mesh filename=package://kdarpa_world/meshes/outdoor_left_wall.STL
- link outdoor_right_wall: geometry collision mesh filename=package://kdarpa_world/meshes/outdoor_right_wall.STL; visual mesh filename=package://kdarpa_world/meshes/outdoor_right_wall.STL
- link second_in_Link: geometry collision mesh filename=package://kdarpa_world/meshes/second_in_Link.STL; visual mesh filename=package://kdarpa_world/meshes/second_in_Link.STL
- link second_out_Link: geometry collision mesh filename=package://kdarpa_world/meshes/second_out_Link.STL; visual mesh filename=package://kdarpa_world/meshes/second_out_Link.STL
- link side_door_link: geometry collision mesh filename=package://kdarpa_world/meshes/side_door_link.STL; visual mesh filename=package://kdarpa_world/meshes/side_door_link.STL
- link stair_1_link: geometry collision mesh filename=package://kdarpa_world/meshes/stair_1_link.STL; visual mesh filename=package://kdarpa_world/meshes/stair_1_link.STL
- link stair_2_Link: geometry collision mesh filename=package://kdarpa_world/meshes/stair_2_Link.STL; visual mesh filename=package://kdarpa_world/meshes/stair_2_Link.STL
- link window_10_link: geometry collision mesh filename=package://kdarpa_world/meshes/window_10_link.STL; visual mesh filename=package://kdarpa_world/meshes/window_10_link.STL
- link window_11_Link: geometry collision mesh filename=package://kdarpa_world/meshes/window_11_Link.STL; visual mesh filename=package://kdarpa_world/meshes/window_11_Link.STL
- link window_12_Link: geometry collision mesh filename=package://kdarpa_world/meshes/window_12_Link.STL; visual mesh filename=package://kdarpa_world/meshes/window_12_Link.STL
- link window_13_Link: geometry collision mesh filename=package://kdarpa_world/meshes/window_13_Link.STL; visual mesh filename=package://kdarpa_world/meshes/window_13_Link.STL
- link window_14_Link: geometry collision mesh filename=package://kdarpa_world/meshes/window_14_Link.STL; visual mesh filename=package://kdarpa_world/meshes/window_14_Link.STL
- link window_15_Link: geometry collision mesh filename=package://kdarpa_world/meshes/window_15_Link.STL; visual mesh filename=package://kdarpa_world/meshes/window_15_Link.STL
- link window_16_Link: geometry collision mesh filename=package://kdarpa_world/meshes/window_16_Link.STL; visual mesh filename=package://kdarpa_world/meshes/window_16_Link.STL
- link window_1_Link: geometry collision mesh filename=package://kdarpa_world/meshes/window_1_Link.STL; visual mesh filename=package://kdarpa_world/meshes/window_1_Link.STL
- link window_2_Link: geometry collision mesh filename=package://kdarpa_world/meshes/window_2_Link.STL; visual mesh filename=package://kdarpa_world/meshes/window_2_Link.STL
- link window_3_Link: geometry collision mesh filename=package://kdarpa_world/meshes/window_3_Link.STL; visual mesh filename=package://kdarpa_world/meshes/window_3_Link.STL
- link window_4_Link: geometry collision mesh filename=package://kdarpa_world/meshes/window_4_Link.STL; visual mesh filename=package://kdarpa_world/meshes/window_4_Link.STL
- link window_5_Link: geometry collision mesh filename=package://kdarpa_world/meshes/window_5_Link.STL; visual mesh filename=package://kdarpa_world/meshes/window_5_Link.STL
- link window_6_Link: geometry collision mesh filename=package://kdarpa_world/meshes/window_6_Link.STL; visual mesh filename=package://kdarpa_world/meshes/window_6_Link.STL
- link window_7_Link: geometry collision mesh filename=package://kdarpa_world/meshes/window_7_Link.STL; visual mesh filename=package://kdarpa_world/meshes/window_7_Link.STL
- link window_8_Link: geometry collision mesh filename=package://kdarpa_world/meshes/window_8_Link.STL; visual mesh filename=package://kdarpa_world/meshes/window_8_Link.STL
- link window_9_Link: geometry collision mesh filename=package://kdarpa_world/meshes/window_9_Link.STL; visual mesh filename=package://kdarpa_world/meshes/window_9_Link.STL

Commit message: px4 sitl simulation added

File: urdf/KDARPA.urdf (robot description, URDF)
Before this commit: robot kdarpa_world, 33 links, 32 joints
Links:
- link stair_3_link: geometry collision mesh filename=package://kdarpa_world/meshes/stair_3_link.STL; visual mesh filename=package://kdarpa_world/meshes/stair_3_link.STL
